File: hardware/kicad/main.kicad_pcb (KiCad board)
At the start: 2 copper layers, 55.6 x 63.5 mm, 85 parts, among them J1 Conn_01x02_Pin, J10 Conn_01x03_Socket, J11 Conn_01x03_Socket, J2 Conn_01x02_Pin, J3 Conn_01x02_Pin, J4 Conn_01x02_Pin, J5 Conn_01x04_Pin, J6 Conn_01x04_Pin, J7 Conn_01x04_Pin, J8 Conn_01x04_Pin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

Commit message: Edit production files
Other:
- board text added: "0.1.6"
- board text removed: "0.9"
Changed lines of the file:
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@@
 		(filling no)
 		(pcbplotparams
-			(layerselection 0x00000000_00000000_55557fdf_ffffffff)
+			(layerselection 0x00000000_00000000_55555555_55555570)
 			(plot_on_all_layers_selection 0x00000000_00000000_00000000_00000000)
 			(disableapertmacros no)
@@
 		)
 	)
-	(gr_text "0.9"
-		(at 136 99.5 0)
+	(gr_text "0.1.6"
+		(at 134.5 100 0)
 		(layer "F.SilkS")
 		(effects
